File: 5strip/ver1.kicad_pcb (KiCad board)
At the start: 2 copper layers, 100 x 50 mm, 57 parts, among them P1 CONN_6, P2 CONN_2, P3 CONN_4X2, P4 CONN_4, P5 CONN_4, P6 CONN_4, P7 CONN_4, P8 CONN_4, Q1 MOSFET_N, Q10 MOSFET_N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

Commit message: Fixed two silk bugs, exported VRML. Bumped version to 0.22
Routing:
- net /driver1/RE: track 41.5 -> 90.5 mm, vias 2 -> 4
- net /MCU_RX: track 35.6 -> 33.6 mm
- net VCC: track 145.4 -> 143.5 mm
- net /NRST: track 42.2 -> 41.5 mm
- net /GPIO6: track 78.9 -> 78.2 mm
Other:
- board text added: "5strip proto v0.22 LED Alert Hackerspace"
- board text removed: "5strip proto v0.21 LED Alert Hackerspace"
